File: dev/dev-board/wrover_peripheral.kicad_sch (KiCad schematic)
At the start: 0 parts

Commit message: making CAD
Parts:
- added AV1: AV-5, easyeda2kicad:CONN-TH_AV-5, symbol easyeda2kicad:AV-5
- added Audio1: PJ-327C-4A, easyeda2kicad:AUDIO-SMD_PJ-327C-4A, symbol easyeda2kicad:PJ-327C-4A
- added C20, C23, C24, C25, C28: 0.1uF, Capacitor_SMD:C_0603_1608Metric, symbol Device:C
- added C21, C22, C26, C27: 10uF, Capacitor_SMD:C_0603_1608Metric, symbol Device:C
- added C29, C30: 2.2uF, Capacitor_SMD:C_0603_1608Metric, symbol Device:C
- added C31, C32: 2.2nF, Capacitor_SMD:C_0603_1608Metric, symbol Device:C
- added J1: Conn_01x04_Pin, Connector_PinHeader_2.54mm:PinHeader_1x04_P2.54mm_Vertical, symbol Connector:Conn_01x04_Pin
- added J2: Conn_01x14_Socket, Connector_PinSocket_2.54mm:PinSocket_1x14_P2.54mm_Vertical, symbol Connector:Conn_01x14_Socket
- added LDO1: ME6211C33M5G-N, easyeda2kicad:SOT-23-5_L3.0-W1.7-P0.95-LS2.8-BL, symbol easyeda2kicad:ME6211C33M5G-N
- added R28, R30, R31, R32: 22, Resistor_SMD:R_0603_1608Metric, symbol Device:R
- added R29, R33: 470, Resistor_SMD:R_0603_1608Metric, symbol Device:R
- added R34: 10K, Resistor_SMD:R_0603_1608Metric, symbol Device:R
- added U13: PCM5102APWR, easyeda2kicad:TSSOP-20_L6.5-W4.4-P0.65-LS6.4-BL, symbol easyeda2kicad:PCM5102APWR
Connections:
- new net: AV1.2, R28.1
- new net: C22.1, C23.1, LDO1.5 (VOUT), U13.1 (CPVDD), U13.8 (AVDD)
- new net: R32.2, U13.15 (LRCK)
- new net: R29.1, U13.7 (OUTR)
- new net: Audio1.3, C32.1, R29.2
- new net: R30.2, U13.13 (BCK)
- new net: R31.2, U13.14 (DIN)
- new net: R34.2, U13.17 (XSMT)
- new net: C25.1, C26.1, U13.18 (LDOO)
- new net: C29.2, U13.2 (CAPP)
- new net: C30.2, U13.3 (CPGND)
- new net: C29.1, U13.4 (CAPM)
- new net: C30.1, U13.5 (VNEG)
- new net: R33.1, U13.6 (OUTL)
- new net: Audio1.2, Audio1.4, C31.1, R33.2
- new net +3V3: C20.1, C21.1, C27.2, C28.2, J2.1 (Pin_1), J2.8 (Pin_8), R34.1, U13.20 (DVDD)
- new net GND: AV1.1, Audio1.1, C20.2, C21.2, C22.2, C23.2, C24.2, C25.2, C26.2, C27.1, C28.1, C31.2, C32.2, J2.2 (Pin_2), LDO1.2 (VSS), U13.10 (DEMP), U13.11 (FLT), U13.12 (SCK), U13.16 (FMT), U13.19 (DGND), U13.9 (AGND)
- new net I2S-BLK: R30.1
- new net I2S-DOUT: R31.1
- new net I2S-WS: R32.1
- new net IO34: J1.3 (Pin_3)
- new net IO35: J1.4 (Pin_4)
- new net IO36: J1.1 (Pin_1)
- new net IO39: J1.2 (Pin_2)
- new net NTSC: R28.2
- new net VSPI-CS: J2.3 (Pin_3)
- new net VSPI-DC: J2.5 (Pin_5)
- new net VSPI-MISO: J2.9 (Pin_9)
- new net VSPI-MOSI: J2.6 (Pin_6)
- new net VSPI-RESET: J2.4 (Pin_4)
- new net VSPI-SCLK: J2.7 (Pin_7)
- new net VSYS: C24.1, LDO1.1 (VIN), LDO1.3 (CE)
- no-connect marks 0 -> 6
Other:
- note added: "ナノ注意"

Commit message: making CAD
Changed lines of the file:
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@@
+	(wire
+		(pts
+			(xy 100.33 92.71) (xy 111.76 92.71)
+		)
+		(stroke
+			(width 0)
+			(type default)
+		)
+	)
 	(wire
 		(pts
@@
 					(unit 1)
 				)
+			)
+		)
+	)
+	(symbol
+		(lib_id "power:GND")
+		(at 100.33 92.71 0)
+		(unit 1)
+		(exclude_from_sim no)
+		(in_bom yes)
+		(on_board yes)
+		(dnp no)
+		(fields_autoplaced yes)
+		(property "Reference" "#PWR040"
+			(at 100.33 99.06 0)
+			(effects
+				(font
+					(size 1.27 1.27)
+				)
+				(hide yes)
+			)
+		)
+		(property "Value" "GND"
+			(at 100.33 97.79 0)
+			(effects
+				(font
+					(size 1.27 1.27)
+				)
+			)
+		)
+		(property "Footprint" ""
+			(at 100.33 92.71 0)
+			(effects
+				(font
+					(size 1.27 1.27)
+				)
+				(hide yes)
+			)
+		)
+		(property "Datasheet" ""
+			(at 100.33 92.71 0)
+			(effects
+				(font
+					(size 1.27 1.27)
+				)
+				(hide yes)
+			)
+		)
+		(property "Description" "Power symbol creates a global label with name \"GND\" , ground"
+			(at 100.33 92.71 0)
+			(effects
+				(font
+					(size 1.27 1.27)
+				)
+				(hide yes)
+			)
+		)
+		(pin "1"
+		)
+		(instances
+			(project ""
+				(path "/211ed859-fe40-48f4-82b7-6e05ddc77423/c5b65813-fac3-4953-8da9-fa09dc19ae64"
+					(reference "#PWR040")
+					(unit 1)
+				)

Commit message: finish cad. 1st step. add symbol,footprint files
Parts:
- added C37: DNP, Capacitor_SMD:C_0603_1608Metric, symbol Device:C
- added J3, J4: DNP Conn_01x02_Pin, Connector_PinHeader_2.54mm:PinHeader_1x02_P2.54mm_Vertical, symbol Connector:Conn_01x02_Pin
- J1: value Conn_01x04_Pin -> DNP Conn_01x04_Pin
- J2: value Conn_01x14_Socket -> DNP Conn_01x14_Socket
Connections:
- net GND: now also C37.2, J3.2 (Pin_2), J4.2 (Pin_2)
- net NTSC: now also J4.1 (Pin_1)
- net VSYS: now also J3.1 (Pin_1)
- net at AV1.2, R28.1: now also C37.1
Other:
- moved on the sheet: R28

Commit message: complete BOM
Parts:
- C20, C23, C24, C25, C28: LCSC Part (none) -> C14663
- C21, C22, C26, C27: LCSC Part (none) -> C19702
- C29, C30: LCSC Part (none) -> C23630
- C31, C32: LCSC Part (none) -> C1604
- R28, R30, R31, R32: LCSC Part (none) -> C23345
- R29, R33: LCSC Part (none) -> C23179
- R34: LCSC Part (none) -> C25804
Changed lines of the file:
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@@
+			)
+		)
+		(property "LCSC Part" "C19702"
+			(at 173.99 46.99 0)
+			(effects
+				(font
+					(size 1.27 1.27)
+				)
+				(hide yes)
 			)
 		)
@@
 			)
 		)
+		(property "LCSC Part" "C23345"
+			(at 106.68 78.74 90)
+			(effects
+				(font
+					(size 1.27 1.27)
+				)
+				(hide yes)
+			)
+		)
 		(pin "1"
 		)
@@
 			)
 		)
+		(property "LCSC Part" "C23179"
+			(at 201.93 76.2 90)
+			(effects
+				(font
+					(size 1.27 1.27)
+				)
+				(hide yes)
+			)
+		)
 		(pin "2"
 		)
@@
 			)
 		)
+		(property "LCSC Part" "C14663"
+			(at 119.38 147.32 0)
+			(effects
+				(font
+					(size 1.27 1.27)
+				)
+				(hide yes)
+			)
+		)
 		(pin "1"
 		)
@@
 			)
 		)
+		(property "LCSC Part" "C25804"
+			(at 146.05 106.68 0)
+			(effects
+				(font
+					(size 1.27 1.27)
+				)
+				(hide yes)
+			)
+		)
 		(pin "2"
 		)
@@
 			)
 		)
+		(property "LCSC Part" "C14663"
+			(at 128.27 46.99 0)
+			(effects
+				(font
+					(size 1.27 1.27)
+				)
+				(hide yes)
+			)
+		)
 		(pin "1"
 		)
@@
 			)
 		)
+		(property "LCSC Part" "C23345"
+			(at 124.46 73.66 90)
+			(effects
+				(font
+					(size 1.27 1.27)
+				)
+				(hide yes)
+			)
+		)
 		(pin "1"
 		)
@@
 			)
 		)
+		(property "LCSC Part" "C23179"
+			(at 210.82 78.74 90)
+			(effects
+				(font
+					(size 1.27 1.27)
+				)
+				(hide yes)
+			)
+		)
 		(pin "1"
 		)
@@
 			)
 		)
+		(property "LCSC Part" "C1604"
+			(at 217.17 85.09 0)
+			(effects
+				(font
+					(size 1.27 1.27)
+				)
+				(hide yes)
+			)
+		)
 		(pin "2"
 		)
@@
 			)
 		)
+		(property "LCSC Part" "C23345"
+			(at 118.11 76.2 90)
+			(effects
+				(font
+					(size 1.27 1.27)
+				)
+				(hide yes)
+			)
+		)
 		(pin "1"
 		)
@@
 		)
 		(property "Description" "Unpolarized capacitor"
+			(at 106.68 147.32 0)
+			(effects
+				(font
+					(size 1.27 1.27)
+				)
+				(hide yes)
+			)
+		)
+		(property "LCSC Part" "C19702"
 			(at 106.68 147.32 0)
 			(effects
@@
 			)
 		)
+		(property "LCSC Part" "C23345"
+			(at 62.23 69.85 90)
+			(effects
+				(font
+					(size 1.27 1.27)
+				)
+				(hide yes)
+			)
+		)
 		(pin "1"
 		)
@@
 			)
 		)
+		(property "LCSC Part" "C19702"
+			(at 111.76 87.63 0)
+			(effects
+				(font
+					(size 1.27 1.27)
+				)
+				(hide yes)
+			)
+		)
 		(pin "2"
 		)
@@
 			)
 		)
+		(property "LCSC Part" "C23630"
+			(at 191.77 87.63 0)
+			(effects
+				(font
+					(size 1.27 1.27)
+				)
+				(hide yes)
+			)
+		)
 		(pin "1"
 		)
@@
 			)
 		)
+		(property "LCSC Part" "C14663"
+			(at 124.46 99.06 0)
+			(effects
+				(font
+					(size 1.27 1.27)
+				)
+				(hide yes)
+			)
+		)
 		(pin "1"
 		)
@@
 			)
 		)
+		(property "LCSC Part" "C23630"
+			(at 180.34 87.63 0)
+			(effects
+				(font
+					(size 1.27 1.27)
+				)
+				(hide yes)
+			)
+		)
 		(pin "2"
 		)
@@
 			)
 		)
+		(property "LCSC Part" "C14663"
+			(at 124.46 87.63 0)
+			(effects
+				(font
+					(size 1.27 1.27)
+				)
+				(hide yes)
+			)
+		)
 		(pin "2"
 		)
@@
 			)
 		)
+		(property "LCSC Part" "C1604"
+			(at 229.87 85.09 0)
+			(effects
+				(font
+					(size 1.27 1.27)
+				)
+				(hide yes)
+			)
+		)
 		(pin "1"
 		)
@@
 			)
 		)
+		(property "LCSC Part" "C14663"
+			(at 185.42 46.99 0)
+			(effects
+				(font
+					(size 1.27 1.27)
+				)
+				(hide yes)
+			)
+		)
 		(pin "2"
 		)
@@
 			(at 111.76 99.06 0)
 			(effects
+				(font
+					(size 1.27 1.27)
+				)
+				(hide yes)
+			)
+		)
+		(property "LCSC Part" "C19702"
+			(at 111.76 99.06 0)
+			(effects

Commit message: update schematics
Parts:
- removed J1: DNP Conn_01x04_Pin, Connector_PinHeader_2.54mm:PinHeader_1x04_P2.54mm_Vertical, symbol Connector:Conn_01x04_Pin
- removed J2: DNP Conn_01x14_Socket, Connector_PinSocket_2.54mm:PinSocket_1x14_P2.54mm_Vertical, symbol Connector:Conn_01x14_Socket
- removed J3, J4: DNP Conn_01x02_Pin, Connector_PinHeader_2.54mm:PinHeader_1x02_P2.54mm_Vertical, symbol Connector:Conn_01x02_Pin
- added J5: Conn_02x10_Odd_Even, Connector_PinHeader_1.00mm:PinHeader_2x10_P1.00mm_Vertical, symbol Connector_Generic:Conn_02x10_Odd_Even
- added TP5: TestPoint, symbol Connector:TestPoint
Connections:
- net +3V3: now also J5.1 (Pin_1)
- net GND: now also J5.12 (Pin_12), J5.19 (Pin_19), J5.2 (Pin_2), J5.3 (Pin_3)
- net IO34: now also J5.8 (Pin_8)
- net IO35: now also J5.10 (Pin_10)
- net IO36: now also J5.4 (Pin_4)
- net IO39: now also J5.6 (Pin_6)
- net NTSC: now also TP5.1
- net VSYS: now also J5.14 (Pin_14)
- new net IO12: J5.5 (Pin_5)
- new net IO13: J5.15 (Pin_15)
- new net IO14: J5.7 (Pin_7)
- new net IO15: J5.9 (Pin_9)
- new net IO26: J5.13 (Pin_13)
- new net IO4: J5.11 (Pin_11)
- new net IO5: J5.17 (Pin_17)
- no-connect marks 6 -> 4
Other:
- moved on the sheet: C20, C21

Commit message: wiring donw. checking DRC
Parts:
- J5: footprint Connector_PinHeader_1.00mm:PinHeader_2x10_P1.00mm_Vertical -> Connector_PinHeader_2.54mm:PinHeader_2x10_P2.54mm_Vertical
- TP5: footprint (none) -> TestPoint:TestPoint_Pad_D1.0mm
Connections:
- net IO34: now also J5.6 (Pin_6); no longer J5.8 (Pin_8)
- net IO35: now also J5.4 (Pin_4); no longer J5.10 (Pin_10)
- net IO36: now also J5.10 (Pin_10); no longer J5.4 (Pin_4)
- net IO39: now also J5.8 (Pin_8); no longer J5.6 (Pin_6)
Changed lines of the file:
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@@
 	(wire
 		(pts
-			(xy 113.03 171.45) (xy 116.84 171.45)
-		)
-		(stroke
-			(width 0)
-			(type default)
-		)
-	)
-	(wire
-		(pts
 			(xy 168.91 86.36) (xy 176.53 86.36)
 		)
@@
 	(wire
 		(pts
-			(xy 113.03 168.91) (xy 116.84 168.91)
-		)
-		(stroke
-			(width 0)
-			(type default)
-		)
-	)
-	(wire
-		(pts
 			(xy 110.49 78.74) (xy 143.51 78.74)
 		)
@@
 	(wire
 		(pts
-			(xy 113.03 163.83) (xy 116.84 163.83)
-		)
-		(stroke
-			(width 0)
-			(type default)
-		)
-	)
-	(wire
-		(pts
 			(xy 73.66 163.83) (xy 86.36 163.83)
 		)
@@
 	(wire
 		(pts
-			(xy 113.03 166.37) (xy 116.84 166.37)
-		)
-		(stroke
-			(width 0)
-			(type default)
-		)
-	)
-	(wire
-		(pts
 			(xy 99.06 73.66) (xy 120.65 73.66)
 		)
@@
 	(hierarchical_label "IO35"
 		(shape output)
-		(at 116.84 171.45 0)
+		(at 113.03 163.83 0)
 		(effects
 			(font
@@
 	(hierarchical_label "IO39"
 		(shape output)
-		(at 116.84 166.37 0)
+		(at 113.03 168.91 0)
 		(effects
 			(font
@@
 	(hierarchical_label "IO36"
 		(shape output)
-		(at 116.84 163.83 0)
+		(at 113.03 171.45 0)
 		(effects
 			(font
@@
 	(hierarchical_label "IO34"
 		(shape output)
-		(at 116.84 168.91 0)
+		(at 113.03 166.37 0)
 		(effects
 			(font
@@
 			)
 		)
-		(property "Footprint" ""
+		(property "Footprint" "TestPoint:TestPoint_Pad_D1.0mm"
 			(at 57.15 132.08 0)
 			(effects
@@
 			)
 		)
-		(property "Footprint" "Connector_PinHeader_1.00mm:PinHeader_2x10_P1.00mm_Vertical"
+		(property "Footprint" "Connector_PinHeader_2.54mm:PinHeader_2x10_P2.54mm_Vertical"
 			(at 105.41 171.45 0)
 			(effects

Commit message: r2 candidate
Parts:
- J5: now not fitted
- TP5: now not fitted; now left out of the parts list
Changed lines of the file:
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@@
 		(unit 1)
 		(exclude_from_sim no)
-		(in_bom yes)
-		(on_board yes)
-		(dnp no)
+		(in_bom no)
+		(on_board yes)
+		(dnp yes)
 		(fields_autoplaced yes)
 		(property "Reference" "TP5"
@@
 		(in_bom yes)
 		(on_board yes)
-		(dnp no)
+		(dnp yes)
 		(property "Reference" "J5"
 			(at 106.68 154.94 0)
