File: dev/dev-board/dev-board.kicad_sch (KiCad schematic)
At the start: 54 parts, among them Q1 BSS138, Q2 BSS138, Q3 BSS138, Q4 BSS138, SW1 TS342A2P, SW2 TS342A2P, SW3 TS342A2P, SW4 TS342A2P, U1 ESP32-WROVER-IE(16MB), U14 CH340C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

Commit message: update for v3r3
Parts:
- removed R12: 100, Resistor_SMD:R_0603_1608Metric, symbol Device:R
- removed RX1, RX2, TX1, TX2: TestPoint, TestPoint:TestPoint_Pad_D1.0mm, symbol Connector:TestPoint
- added R42: 0, Resistor_SMD:R_0603_1608Metric, symbol Device:R
- added SW9: GT-TC018A-H0375-L1, easyeda2kicad:SW-SMD_L4.7-W3.5-P3.35-EH, symbol easyeda2kicad:GT-TC018A-H0375-L1
Connections:
- net GND: now also SW9.1, SW9.3, SW9.4
- net S3-EN: now also SW9.2
- net S3-ResetSub: now also R42.2
- net WR-EN: now also R42.1
