File: dev/dev-board/dev-board.kicad_pcb (KiCad board)
At the start: 4 copper layers, 90 x 70 mm, 132 parts, among them J1 Conn_01x03_Pin, J2 Conn_01x02_Socket, J5 Conn_02x10_Odd_Even, Q1 BSS138, Q2 BSS138, Q3 BSS138, Q4 BSS138, SW9 GT-TC018A-H0375-L1, U1 ESP32-WROVER-IE(16MB), U10 TPS2065CDBV, U11 PESD5V0U2BT, U12 PESD5V0S1BA_C5261083, U13 PCM5102APWR, U14 CH340C, U15 RX8900CE_UB0, U16 PESD5V0U2BT, U2 ESP32-S3-WROOM-1(N16R8), U3 CH340C, U4 TPS2065CDBV, U5 AP7361C-33E, U6 PESD5V0U2BT, U7 PESD5V0S1BA_C5261083, U8 ZX-HY2.0-4PWZ, U9 ZX-HY2.0-4PWZ

Commit message: v3 dev r3 candidate
Routing:
- net GND: track 241.2 -> 242.7 mm, vias 272 -> 273
Changed lines of the file:
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@@
 	)
 	(segment
-		(start 77.283004 9.761066)
-		(end 77.283004 9.488934)
-		(width 0.2)
-		(layer "F.Cu")
-		(net 3)
-	)
-	(segment
 		(start 53.191938 6.9975)
 		(end 53.561938 6.9975)
@@
 	)
 	(segment
+		(start 84.334438 58.25)
+		(end 84.521938 58.25)
+		(width 0.2)
+		(layer "F.Cu")
+		(net 3)
+	)
+	(segment
 		(start 40.746938 13.25)
 		(end 40.746938 12.725)
@@
 	)
 	(segment
-		(start 79.229045 11.707107)
-		(end 77.283004 9.761066)
-		(width 0.2)
-		(layer "F.Cu")
-		(net 3)
-	)
-	(segment
 		(start 83.024438 10.4975)
 		(end 83.024438 9.67)
@@
 	)
 	(segment
+		(start 82.584438 56.5)
+		(end 84.334438 58.25)
+		(width 0.2)
+		(layer "F.Cu")
+		(net 3)
+	)
+	(segment
 		(start 84.941938 9.67)
 		(end 85.271938 10)
@@
 	)
 	(segment
+		(start 77.896938 10.375)
+		(end 79.229045 11.707107)
+		(width 0.2)
+		(layer "F.Cu")
+		(net 3)
+	)
+	(segment
 		(start 81.421938 19.85)
 		(end 81.521938 19.75)
@@
 	)
 	(via
+		(at 84.521938 58.25)
+		(size 0.6)
+		(drill 0.3)
+		(layers "F.Cu" "B.Cu")
+		(free yes)
+		(net 3)
+	)
+	(via
 		(at 64.521938 47.5)
 		(size 0.6)
@@
 	)
 	(via
-		(at 77.283004 9.488934)
+		(at 77.896938 10.375)
 		(size 0.6)
 		(drill 0.3)
@@
 	)
 	(segment
+		(start 17.271938 61.6375)
+		(end 16.310438 62.599)
+		(width 0.2)
+		(layer "F.Cu")
+		(net 64)
+	)
+	(segment
 		(start 54.021938 55.25)
 		(end 56.521938 55.25)
@@
 	)
 	(segment
-		(start 63.271938 43.258)
-		(end 64.109938 42.42)
+		(start 16.310438 62.599)
+		(end 9.120938 62.599)
 		(width 0.2)
 		(layer "F.Cu")
@@
 	)
 	(segment
-		(start 4.510938 58.211)
-		(end 5.221938 57.5)
+		(start 63.271938 43.258)
+		(end 64.109938 42.42)
 		(width 0.2)
 		(layer "F.Cu")
@@
 	)
 	(segment
+		(start 4.510938 60.049534)
+		(end 4.510938 58.211)
+		(width 0.2)
+		(layer "F.Cu")
+		(net 64)
+	)
+	(segment
 		(start 18.771938 63.1375)
 		(end 18.771938 64.5)
@@
 	)
 	(segment
+		(start 9.120938 62.599)
+		(end 8.021938 61.5)
+		(width 0.2)
+		(layer "F.Cu")
+		(net 64)
+	)
+	(segment
+		(start 4.822404 60.361)
+		(end 4.510938 60.049534)
+		(width 0.2)
+		(layer "F.Cu")
+		(net 64)
+	)
+	(segment
 		(start 17.521938 61.8875)
 		(end 18.771938 63.1375)
@@
 	)
 	(segment
-		(start 16.310438 62.599)
-		(end 7.060404 62.599)
+		(start 6.521938 61.5)
+		(end 5.382938 60.361)
 		(width 0.2)
 		(layer "F.Cu")
@@
 	)
 	(segment
-		(start 17.521938 59.075)
-		(end 17.521938 61.8875)
+		(start 5.382938 60.361)
+		(end 4.822404 60.361)
 		(width 0.2)
 		(layer "F.Cu")
@@
 	)
 	(segment
-		(start 4.510938 60.049534)
-		(end 4.510938 58.211)
+		(start 17.521938 59.075)
+		(end 17.521938 61.8875)
 		(width 0.2)
 		(layer "F.Cu")
@@
 	)
 	(segment
-		(start 18.771938 64.5)
-		(end 20.021938 65.75)
+		(start 8.021938 61.5)
+		(end 6.521938 61.5)
 		(width 0.2)
 		(layer "F.Cu")
@@
 	)
 	(segment
-		(start 7.060404 62.599)
-		(end 4.510938 60.049534)
+		(start 4.510938 58.211)
+		(end 5.221938 57.5)
 		(width 0.2)
 		(layer "F.Cu")
@@
 	)
 	(segment
-		(start 56.521938 55.25)
-		(end 62.420938 49.351)
+		(start 18.771938 64.5)
+		(end 20.021938 65.75)
 		(width 0.2)
 		(layer "F.Cu")
@@
 	)
 	(segment
-		(start 17.271938 61.6375)
-		(end 16.310438 62.599)
+		(start 56.521938 55.25)
+		(end 62.420938 49.351)
 		(width 0.2)
 		(layer "F.Cu")

Commit message: v3 dev r3 candidate2
Parts:
- D4: renamed from ERR1; footprint LED_SMD:LED_0805_2012Metric -> LED_SMD:LED_0603_1608Metric
- renumbered STAT1 to D1, JTAG to P1, S3-IO0 to SW1, WR-IO0 to SW2, S3-EN to SW3, WR-EN to SW4, UP to SW5, CANCEL to SW6, Enter to SW7, DOWN to SW8
Routing:
- net GND: track 242.7 -> 242.6 mm, vias 273 -> 280
Other:
- board text added: "Cancel"
- board text added: "Down"
- board text added: "Enter"
- board text added: "RW-IO0"
- board text added: "S3-EN"
- board text added: "S3-IO0"
- board text added: "Up"
- board text added: "WR-EN"
